File: UPDI-USB-SERIAL.kicad_pcb (KiCad board)
At the start: 2 copper layers, 15.2 x 40.6 mm, 56 parts, among them J1 USB-C_16Pins, J2 2.54mm 1x6, Q1 BSS138DW, Q2 BSS138DW, SW1 TS-107A, U1 ATMEGA328P-MU, U2 ME6216A33XG, U3 CP2105, Y1 X322516MOB4SI

Commit message: v2.00
Parts:
- removed C10: 100nF, RocketScreamKiCadLib:C_0603
- removed C13: 10uF 16V X5R, RocketScreamKiCadLib:C_0603
- removed the C5 at (144.8, 99.8)
- removed the C8 at (144.8, 93.7)
- removed the C9 at (134.0, 97.7)
- removed TP3, TP4, TP5, TP6: TEST-PAD, RocketScreamKiCadLib:TEST-PAD-1.5MM
- removed Y1: X322516MOB4SI, RocketScreamKiCadLib:CRYSTAL-3225-4P
- added D4: Yellow, RocketScreamKiCadLib:LED_0603, F.Cu at (145.2, 93.7)
- added L2: BLM18KG221SN1D, RocketScreamKiCadLib:I_0603, F.Cu at (135.3, 98.7)
- added M1: FIDUCIAL, RocketScreamKiCadLib:FIDUCIAL-0.5MM_CROSS, F.Cu at (134.4, 120.8)
- added M2: FIDUCIAL, RocketScreamKiCadLib:FIDUCIAL-0.5MM_CROSS, F.Cu at (145.0, 120.8)
- added M3: FIDUCIAL, RocketScreamKiCadLib:FIDUCIAL-0.5MM_CROSS, F.Cu at (133.4, 82.4)
- added M4: FIDUCIAL, RocketScreamKiCadLib:FIDUCIAL-0.5MM_CROSS, F.Cu at (146.1, 82.4)
- added R14: 5K1, RocketScreamKiCadLib:R_0603, F.Cu at (145.2, 95.3)
- LOGO1: renamed from LOGO2; footprint RocketScreamKiCadLib:LOGO-ROCKET-SCREAM_Horizontal_XXSmall -> RocketScreamKiCadLib:LOGO-ROCKET-SCREAM_Horizontal_XSmall
- U1: value ATMEGA328P-MU -> CH342F; footprint RocketScreamKiCadLib:QFN-32_5x5mm_Pitch0.5mm -> RocketScreamKiCadLib:QFN-24_4x4mm_Pitch0.5mm
- U3: value CP2105 -> ATMEGA808-MU; footprint RocketScreamKiCadLib:QFN-24_4x4mm_Pitch0.5mm -> RocketScreamKiCadLib:QFN-32_5x5mm_Pitch0.5mm
- moved LOGO3 16.6 mm to (142.2, 112.0)
- moved D3 12.6 mm to (146.1, 115.7)
- moved D2 12.4 mm to (133.5, 115.7)
- moved R9 10.2 mm to (145.0, 107.2), turned to 180 degrees
- moved R11 9.84 mm to (145.0, 105.6), turned to 180 degrees
- moved R6 9.76 mm to (135.2, 110.5), turned to 90 degrees
- moved R8 9.26 mm to (136.8, 111.1), turned to 90 degrees
- moved C9 9.01 mm to (136.8, 98.7), turned to -90 degrees
- moved TP2 8.63 mm to (140.0, 99.1)
- moved TP1 8.63 mm to (140.0, 101.6)
- moved U3 8.00 mm to (141.9, 99.6), turned to 180 degrees
- moved U1 7.85 mm to (140.4, 107.6), turned to 90 degrees
- moved LOGO1 6.30 mm to (139.7, 93.5)
- moved C4 4.36 mm to (139.7, 103.9), turned to 0 degrees
- moved JP4 4.36 mm to (139.7, 103.9), turned to 0 degrees
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- renumbered C4 to C1, C3 to C2, C14 to C3, C11 to C4, C1 to C5, C2 to C6, C12 to C7, C6 to C8, C7 to C9, D3 to D1, D1 to D2, D2 to D3, J2 to J1, J1 to J2, JP3 to JP2, JP4 to JP3, JP2 to JP4, LOGO1 to LOGO2, R6 to R1, R9 to R10, R1 to R11, R8 to R13, R14 to R15, R10 to R16, R7 to R2, R11 to R3, R5 to R4, R15 to R5, R4 to R6, R13 to R7, R3 to R8, R2 to R9
Connections:
- C2 pad 1: 3V3 -> 5V
- C3 pad 1: Net-(C14-Pad1) -> Net-(C3-Pad1)
- C4 pad 2: /~{RESET} -> /RST_HOST
- C8 pad 1: 3V3 -> 5V
- C9 pad 1: 3V3 -> Net-(C9-Pad1)
- D1 pad 1: 3V3 -> 5V
- D1 pad 2: /~{RESET} -> /RST_HOST
- D2 pad 1: 3V3 -> 5V
- D2 pad 2: 3V3 -> 5V
- D3 pad 1: 3V3 -> 5V
- D3 pad 2: 3V3 -> 5V
- J1 pad 5: /UPDI -> /UPDI_TGT
- J2 pad A8: Net-(J1-PadA8) -> unconnected-(J2-PadA8)
- J2 pad B8: Net-(J1-PadB8) -> unconnected-(J2-PadB8)
- JP2 pad 1: /~{RTS} -> /DTR
- JP2 pad 2: /~{RTS1} -> /DTR1
- JP4 pad 2: /~{RTS0} -> /DTR0
- Q1 pad 1: /D6 -> /UPDI_TGT
- Q1 pad 2: 3V3 -> VCC
- Q1 pad 3: /TXD -> /TXD1
- Q1 pad 4: /TXD1 -> /TXD
- Q1 pad 5: 3V3 -> VCC
- Q1 pad 6: /UPDI -> /D8
- Q2 pad 1: /RXD1 -> /RXD
- Q2 pad 2: 3V3 -> VCC
- Q2 pad 3: /RST -> /DTR
- Q2 pad 4: /~{RTS} -> /RST
- Q2 pad 5: 3V3 -> VCC
- Q2 pad 6: /RXD -> /RXD1
- R10 pad 1: /TXD -> /TXD1
- R10 pad 2: VCC -> 5V
- R11 pad 2: Net-(R1-Pad2) -> /TXD1
- R12 pad 1: /RXD -> /RXD1
- R12 pad 2: VCC -> 5V
- R13 pad 1: /RXD1 -> /RXD
- R13 pad 2: 3V3 -> VCC
- R15 pad 1: /~{RTS} -> /RST
- R15 pad 2: 3V3 -> VCC
- R16 pad 1: /RST -> /DTR
- R16 pad 2: VCC -> 5V
- R3 pad 1: /UPDI -> /D8
- R3 pad 2: VCC -> 5V
- R4 pad 1: /D6 -> /UPDI_TGT
- R4 pad 2: 3V3 -> VCC
- R5 pad 1: /~{RESET} -> /RST_HOST
- R5 pad 2: 3V3 -> 5V
- R6 pad 2: Net-(R4-Pad2) -> /RXD0
- R7 pad 1: /TXD1 -> /TXD
- R7 pad 2: 3V3 -> VCC
- R8 pad 2: Net-(R3-Pad2) -> /TXD0
- R9 pad 2: Net-(R2-Pad2) -> /RXD1
- SW1 pad 1: /~{RESET} -> /RST_HOST
- U1 pad 1: Net-(U1-Pad1) -> unconnected-(U1-Pad1)
- U1 pad 10: /D6 -> unconnected-(U1-Pad10)
- U1 pad 11: Net-(U1-Pad11) -> unconnected-(U1-Pad11)
- U1 pad 12: Net-(U1-Pad12) -> /RXD1
- U1 pad 13: Net-(U1-Pad13) -> /TXD1
- U1 pad 14: Net-(U1-Pad14) -> unconnected-(U1-Pad14)
- U1 pad 15: /D11 -> /DTR1
- U1 pad 16: /D12 -> unconnected-(U1-Pad16)
- U1 pad 17: /D13 -> unconnected-(U1-Pad17)
- U1 pad 18: 3V3 -> unconnected-(U1-Pad18)
- U1 pad 19: Net-(U1-Pad19) -> unconnected-(U1-Pad19)
- U1 pad 2: Net-(U1-Pad2) -> GND
- U1 pad 20: AREF -> /RXD0
- U1 pad 21: GND -> /TXD0
- U1 pad 22: Net-(U1-Pad22) -> unconnected-(U1-Pad22)
- U1 pad 23: Net-(U1-Pad23) -> /DTR0
- U1 pad 24: Net-(U1-Pad24) -> unconnected-(U1-Pad24)
- U1 pad 25: Net-(U1-Pad25) -> GND
- U1 pad 3: GND -> /D+
- U1 pad 4: 3V3 -> /D-
- U1 pad 5: GND -> 5V
- U1 pad 6: 3V3 -> Net-(C3-Pad1)
- U1 pad 7: Net-(C5-Pad1) -> 5V
- U1 pad 8: Net-(C8-Pad1) -> 5V
- U1 pad 9: Net-(U1-Pad9) -> unconnected-(U1-Pad9)
- U3 pad 1: Net-(U3-Pad1) -> unconnected-(U3-Pad1)
- U3 pad 10: Net-(U3-Pad10) -> unconnected-(U3-Pad10)
- U3 pad 11: /~{RTS0} -> unconnected-(U3-Pad11)
- U3 pad 12: /D1 -> unconnected-(U3-Pad12)
- U3 pad 13: /D0 -> unconnected-(U3-Pad13)
- U3 pad 14: Net-(R4-Pad2) -> unconnected-(U3-Pad14)
- U3 pad 15: Net-(R3-Pad2) -> unconnected-(U3-Pad15)
- U3 pad 16: Net-(C13-Pad1) -> unconnected-(U3-Pad16)
- U3 pad 17: Net-(U3-Pad17) -> unconnected-(U3-Pad17)
- U3 pad 18: Net-(U3-Pad18) -> Net-(C9-Pad1)
- U3 pad 19: /~{RTS1} -> GND
- U3 pad 2: GND -> unconnected-(U3-Pad2)
- U3 pad 20: /RXD1 -> unconnected-(U3-Pad20)
- U3 pad 21: /TXD1 -> unconnected-(U3-Pad21)
- U3 pad 22: Net-(U3-Pad22) -> unconnected-(U3-Pad22)
- U3 pad 23: Net-(R2-Pad2) -> unconnected-(U3-Pad23)
- U3 pad 24: Net-(R1-Pad2) -> unconnected-(U3-Pad24)
- U3 pad 25: GND -> unconnected-(U3-Pad25)
- U3 pad 3: /D+ -> unconnected-(U3-Pad3)
- U3 pad 4: /D- -> unconnected-(U3-Pad4)
- U3 pad 5: 3V3 -> /D7
- U3 pad 6: Net-(C14-Pad1) -> /D8
- U3 pad 7: 5V -> unconnected-(U3-Pad7)
- U3 pad 8: 5V -> unconnected-(U3-Pad8)
- U3 pad 9: Net-(U3-Pad9) -> unconnected-(U3-Pad9)
Routing:
- net 3V3: track 118.3 -> 14.3 mm, vias 8 -> 1
- net 5V: track 21.3 -> 94.5 mm, vias 2 -> 11
- net /~{RESET}: track 30.5 -> 0.00 mm, vias 5 -> 0
- net /DTR: track 0.00 -> 19.5 mm, vias 0 -> 3
- net /~{RTS}: track 19.0 -> 0.00 mm, vias 1 -> 0
- net /D6: track 16.9 -> 0.00 mm, vias 2 -> 0
- net /RST_HOST: track 0.00 -> 15.8 mm, vias 0 -> 2
- net /DTR0: track 0.00 -> 15.8 mm, vias 0 -> 1
- net /TXD0: track 0.00 -> 14.0 mm, vias 0 -> 2
- net /RXD0: track 0.00 -> 13.8 mm, vias 0 -> 2
- net /D8: track 0.00 -> 12.0 mm
- net /UPDI: track 8.24 -> 0.00 mm, vias 1 -> 0
- net /D13: track 7.77 -> 0.00 mm, vias 1 -> 0
- net Net-(R3-Pad2): track 7.14 -> 0.00 mm, vias 2 -> 0
- net Net-(R4-Pad2): track 6.78 -> 0.00 mm, vias 2 -> 0
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- removed copper zone on F.Cu, net 3V3
- removed copper zone on F.Cu, net 5V
Other:
- board text added: "2022-07"
- board text added: "DTR"
- board text added: "HOST UPDI"
- board text added: "Serial"
- board text added: "UPDI-USB-SERIAL 2v00"
- board text added: "USB"
- board text removed: "2020-07"
- board text removed: "AVR-ISP"
- board text removed: "RTS"
- board text removed: "UPDI-USB-SERIAL 1v00"
