File: UPDI-USB-SERIAL.kicad_sch (KiCad schematic)
At the start: 56 parts

Commit message: v2.00
Parts:
- removed C10, C13, C5, C8, C9: (no value), symbol RocketScreamKiCadLib:CAPACITOR-CERAMIC
- removed TP3, TP4, TP5, TP6: (no value), symbol RocketScreamKiCadLib:TEST-PAD
- removed U1: (no value), symbol RocketScreamKiCadLib:ATMEGA328P-MU
- removed U3: (no value), symbol RocketScreamKiCadLib:CP2105
- removed Y1: (no value), symbol RocketScreamKiCadLib:CRYSTAL_4Pins
- added D4: Yellow, RocketScreamKiCadLib:LED_0603, symbol RocketScreamKiCadLib:LED-SINGLE
- added L2: BLM18KG221SN1D, RocketScreamKiCadLib:I_0603, symbol RocketScreamKiCadLib:INDUCTOR
- added M1, M2, M3, M4: FIDUCIAL, RocketScreamKiCadLib:FIDUCIAL-0.5MM_CROSS, symbol RocketScreamKiCadLib:FIDUCIAL
- added R14: 5K1, RocketScreamKiCadLib:R_0603, symbol RocketScreamKiCadLib:RESISTOR
- added U1: CH342F, RocketScreamKiCadLib:QFN-24_4x4mm_Pitch0.5mm, symbol RocketScreamKiCadLib:CH342F
- added U3: ATMEGA808-MU, RocketScreamKiCadLib:QFN-32_5x5mm_Pitch0.5mm, symbol RocketScreamKiCadLib:ATMEGAx808-Mx
- C1: renamed from C4; value (none) -> 10uF 16V X5R; footprint (none) -> RocketScreamKiCadLib:C_0603
- C2: renamed from C3; value (none) -> 100nF; footprint (none) -> RocketScreamKiCadLib:C_0603
- C3: renamed from C14; value (none) -> 10uF 16V X5R; footprint (none) -> RocketScreamKiCadLib:C_0603
- C4: renamed from C11; value (none) -> 100nF; footprint (none) -> RocketScreamKiCadLib:C_0603
- C5: renamed from C1; value (none) -> 10uF 16V X5R; footprint (none) -> RocketScreamKiCadLib:C_0603
- C6: renamed from C2; value (none) -> 100nF; footprint (none) -> RocketScreamKiCadLib:C_0603
- C7: renamed from C12; value (none) -> 10uF 16V X5R; footprint (none) -> RocketScreamKiCadLib:C_0603
- C8: renamed from C6; value (none) -> 100nF; footprint (none) -> RocketScreamKiCadLib:C_0603
- C9: renamed from C7; value (none) -> 100nF; footprint (none) -> RocketScreamKiCadLib:C_0603
- D1: renamed from D3; value (none) -> 1N4148WS; footprint (none) -> RocketScreamKiCadLib:SOD-323
- D2: renamed from D1; value (none) -> 18-225A/R6GHC-A01/3T; footprint (none) -> RocketScreamKiCadLib:LED-18-225
- D3: renamed from D2; value (none) -> 18-225A/R6GHC-A01/3T; footprint (none) -> RocketScreamKiCadLib:LED-18-225
- F1: value (none) -> MF-FSMF050X-2; footprint (none) -> RocketScreamKiCadLib:MF-FSMF
- J1: renamed from J2; value (none) -> 2.54mm 1x6; footprint (none) -> RocketScreamKiCadLib:RCP_1x6_Pitch2.54mm_RightAngle
- J2: renamed from J1; value (none) -> USB-C_16Pins; footprint (none) -> RocketScreamKiCadLib:TYPE-C16PIN
- JP1: value (none) -> JUMPER-2-WAY; footprint (none) -> RocketScreamKiCadLib:JUMPER-2-WAY-SMD
- JP2: renamed from JP3; value (none) -> JUMPER-1-WAY; footprint (none) -> RocketScreamKiCadLib:JUMPER-1-WAY-SMD
- JP3: renamed from JP4; value (none) -> JUMPER-2-WAY; footprint (none) -> RocketScreamKiCadLib:JUMPER-2-WAY-SMD
- JP4: renamed from JP2; value (none) -> JUMPER-1-WAY; footprint (none) -> RocketScreamKiCadLib:JUMPER-1-WAY-SMD
- L1: value (none) -> BLM18KG221SN1D; footprint (none) -> RocketScreamKiCadLib:I_0603
- LOGO1: renamed from LOGO2; value (none) -> LOGO-ROCKET-SCREAM-HORIZONTAL; footprint (none) -> RocketScreamKiCadLib:LOGO-ROCKET-SCREAM_Horizontal_XSmall
- LOGO2: renamed from LOGO1; value (none) -> LOGO-OSHW; footprint (none) -> RocketScreamKiCadLib:LOGO-OSHW_XSmall
- LOGO3: value (none) -> LOGO-KICAD; footprint (none) -> RocketScreamKiCadLib:LOGO-KICAD_XXXSmall
- Q1, Q2: value (none) -> BSS138DW; footprint (none) -> RocketScreamKiCadLib:SOT-363_Diodes_Inc
- R1: renamed from R6; value (none) -> 5K1; footprint (none) -> RocketScreamKiCadLib:R_0603
- R10: renamed from R9; value (none) -> 10K; footprint (none) -> RocketScreamKiCadLib:R_0603
- R11: renamed from R1; value (none) -> 5K1; footprint (none) -> RocketScreamKiCadLib:R_0603
- R12: value (none) -> 10K; footprint (none) -> RocketScreamKiCadLib:R_0603
- R13: renamed from R8; value (none) -> 10K; footprint (none) -> RocketScreamKiCadLib:R_0603
- R15: renamed from R14; value (none) -> 10K; footprint (none) -> RocketScreamKiCadLib:R_0603
- R16: renamed from R10; value (none) -> 10K; footprint (none) -> RocketScreamKiCadLib:R_0603
- R2: renamed from R7; value (none) -> 5K1; footprint (none) -> RocketScreamKiCadLib:R_0603
- R3: renamed from R11; value (none) -> 100K; footprint (none) -> RocketScreamKiCadLib:R_0603
- R4: renamed from R5; value (none) -> 100K; footprint (none) -> RocketScreamKiCadLib:R_0603
- R5: renamed from R15; value (none) -> 10K; footprint (none) -> RocketScreamKiCadLib:R_0603
- R6: renamed from R4; value (none) -> 5K1; footprint (none) -> RocketScreamKiCadLib:R_0603
- R7: renamed from R13; value (none) -> 10K; footprint (none) -> RocketScreamKiCadLib:R_0603
- R8: renamed from R3; value (none) -> 5K1; footprint (none) -> RocketScreamKiCadLib:R_0603
- R9: renamed from R2; value (none) -> 5K1; footprint (none) -> RocketScreamKiCadLib:R_0603
- SW1: value (none) -> TS-107A; footprint (none) -> RocketScreamKiCadLib:TS-107A
- TP1, TP2: value (none) -> TEST-PAD; footprint (none) -> RocketScreamKiCadLib:TEST-PAD-1.5MM
- U2: value (none) -> ME6216A33XG; footprint (none) -> RocketScreamKiCadLib:SOT-23
Connections:
- net D13 is gone; now on net GND: TP2.1
- net 3V3: no longer C2.1, C8.1, C9.1, D1.1 (K), D2.1 (A), D2.2 (A), D3.1 (A), D3.2 (A), Q1.2 (G2), Q1.5 (G1), Q2.2 (G2), Q2.5 (G1), R13.2, R15.2, R4.2, R5.2, R7.2
- net 5V: now also C2.1, C8.1, D1.1 (K), D2.1 (A), D2.2 (A), D3.1 (A), D3.2 (A), R10.2, R12.2, R16.2, R3.2, R5.2, L2.2, U1.5 (VIO), U1.7 (VDD5), U1.8 (VBUS), U3.28 (VDD)
- net D+: now also U1.3 (UD+)
- net D-: now also U1.4 (UD-)
- net GND: now also D4.1 (K), U1.2 (GND), U1.25 (GND), U3.19 (GND), U3.29 (GND), U3.33 (GND)
- net RST: now also Q2.4 (S1), R15.1; no longer Q2.3 (D1), R16.1
- net RXD: now also Q2.1 (S2), R13.1; no longer Q2.6 (D2), R12.1
- net RXD1: now also Q2.6 (D2), R12.1, R9.2, U1.12 (RXD1); no longer Q2.1 (S2), R13.1
- net TXD: now also Q1.4 (S1), R7.1; no longer Q1.3 (D1), R10.1
- net TXD1: now also Q1.3 (D1), R10.1, R11.2, U1.13 (TXD1); no longer Q1.4 (S1), R7.1
- net VCC: now also Q1.2 (G2), Q1.5 (G1), Q2.2 (G2), Q2.5 (G1), R13.2, R15.2, R4.2, R7.2; no longer R10.2, R12.2, R16.2, R3.2
- net RXD0: now reaches R6.2
- net RXD0: now also U1.20 (RXD0), U3.30 (PA0/EXTCLK)
- net TXD0: now reaches R8.2
- net TXD0: now also U1.21 (TXD0), U3.31 (PA1)
- net at C3.1: now also U1.6 (V3)
- net D12 renamed UPDI_HOST
- net UPDI_HOST: now also U3.27 (UPDI)
- net D6 renamed UPDI_TGT
- net UPDI_TGT: now also J1.5
- net UPDI renamed D8
- net D8: now also U3.6 (PC0); no longer J1.5
- net ~{RESET} renamed RST_HOST
- net RST_HOST: now also U3.26 (PF6)
- net ~{RTS0} renamed DTR0
- net DTR0: now also U1.23 (DTR0)
- net ~{RTS1} renamed DTR1
- net DTR1: now also U1.15 (DTR1)
- removed net ~{RTS}: JP2.1, Q2.4 (S1), R15.1
- new net: C9.1, L2.1, U3.18 (AVDD)
- new net: D4.2 (A), R14.1
- new net D7: R14.2, U3.5 (PA7)
- new net DTR: JP2.1, Q2.3 (D1), R16.1
- no-connect marks 24 -> 35
Other:
- note added: "ATmega808"
- note added: "Auto reset on ATMega808"
- note added: "Fiducials"
- note added: "Host UPDI Test Points"
- note added: "Indicator LEDs"
- note added: "Select board variant as: -ATmega808/ATmega4808 32-pin standard -internal 16MHz oscillator -UART0 default pins bootloader"
- note removed: "16MHz"
- note removed: "ATmega328P"
- note removed: "Auto reset on ATMega328P"
- note removed: "ISP Test Points"
- note removed: "Select board variant as "Arduino Uno""
- moved on the sheet: C4, C8, C9, D1, D2, D3, J1, JP4, Q1, Q2, R10, R11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
